File: hardware/bms_10s.kicad_pcb (KiCad board)
At the start: 2 copper layers, 100 x 40 mm, 129 parts, among them J1 BAL, J10 Conn_01x05, J11 Conn_01x03, J2 THERM_2, J4 THERM_1, J5 BAT_NEG_IN, J6 PACK-, J7 Conn_01x04, Q1 NTR3C21NZ, Q10 NTR3C21NZ, Q11 BUK762R6-60E, Q12 BUK762R6-60E, Q13 SI2337DS-T1-E3, Q2 NTR3C21NZ, Q3 NTR3C21NZ, Q4 NTR3C21NZ, Q5 NTR3C21NZ, Q6 NTR3C21NZ, Q7 NTR3C21NZ, Q8 NTR3C21NZ, Q9 NTR3C21NZ, U1 bq7693002DBT, U2 BUK9Y43-60E, U3 STM32L031F4Px, U4 ISO7021

Commit message: PCB layout done
Signed-off-by: Ene Alexandru <ene.alexandru@gmail.com>
Parts:
- C16, R1, R54: moved to B.Cu
- moved R54 4.77 mm to (27.0, 52.5), turned to 180 degrees
- moved R1 1.75 mm to (30.3, 52.3)
- moved C16 1.37 mm to (30.3, 56.1), turned to 270 degrees
Routing:
- net /input/B1: track 22.8 -> 28.3 mm
- net /bq/TS1: track 57.1 -> 54.4 mm
- net GND: track 23.3 -> 22.0 mm
Other:
- board text added: "B0"
- board text added: "B1"
- board text added: "B10"
- board text added: "B2"
- board text added: "B3"
- board text added: "B4"
- board text added: "B5"
- board text added: "B6"
- board text added: "B7"
- board text added: "B8"
- board text added: "B9"
- board text added: "BATT_NEG"
- board text added: "BMS BOOT"
- board text added: "BOOT0"
- board text added: "ISOL_GND"
- board text added: "ISOL_RX"
- board text added: "ISOL_TX"
- board text added: "ISOL_VCC"
- board text added: "PACK_NEG POWER OUT"
- board text added: "SWCLK"
- board text added: "SWDIO"
- board text added: "TS1"
- board text added: "TS2"
- board text added: "UART2_RX"
- board text added: "UART2_TX"
- board text added: "~NRST"
